File: USB3300.kicad_pcb (KiCad board)
At the start: 2 copper layers, 49 parts, among them J1 SWD, J2 Conn_01x02_Pin, J3 USB_C_Receptacle_USB2.0_14P, SW1 SW_SPDT, U1 USB3300-EZK, U2 STM32F405RGT6, U3 XC6206PxxxMR, U4 SRV05-4, Y1 16MHz, Y2 24MHz

Commit message: work on pcb
Parts:
- moved J3 61.6 mm to (159.5, 146.3), turned to 0 degrees
- moved F1 59.3 mm to (149.8, 142.4)
- moved C15 56.0 mm to (149.9, 139.7)
- moved R9 51.4 mm to (149.9, 137.7)
- moved FB1 48.3 mm to (144.3, 139.2), turned to 90 degrees
- moved SW1 39.0 mm to (171.9, 108.2), turned to 90 degrees
- moved C23 37.0 mm to (149.9, 135.1)
- moved U3 33.1 mm to (149.7, 132.0), turned to 180 degrees
- moved R10 32.0 mm to (138.7, 119.9), turned to 90 degrees
- moved R1 26.2 mm to (167.1, 109.2), turned to 180 degrees
- moved C14 26.1 mm to (175.2, 128.2), turned to 180 degrees
- moved C13 24.6 mm to (178.3, 131.6), turned to 90 degrees
- moved Y2 24.0 mm to (175.3, 131.6), turned to 90 degrees
- moved J1 19.5 mm to (144.3, 126.1)
- moved L1 15.9 mm to (150.4, 119.4)
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Routing:
- net ULPI_STP: track 0.00 -> 40.3 mm
- net ULPI_D7: track 0.00 -> 37.2 mm
- net ULPI_DIR: track 0.00 -> 35.4 mm
- net ULPI_NXT: track 0.00 -> 29.5 mm
- net ULPI_D6: track 0.00 -> 14.1 mm
- net ULPI_D5: track 0.00 -> 12.4 mm
- net ULPI_D0: track 0.00 -> 10.2 mm
- net ULPI_D3: track 0.00 -> 9.48 mm
- net ULPI_D4: track 0.00 -> 9.48 mm
- net GND: track 0.00 -> 9.33 mm
- net ULPI_D1: track 0.00 -> 9.27 mm
- net ULPI_D2: track 0.00 -> 9.27 mm
- net +3V3: track 0.00 -> 8.41 mm
- net USART1_TX: track 0.00 -> 7.79 mm
- net USART1_RX: track 0.00 -> 6.95 mm
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